Commit message: Parte1 Notion. Rviz

File: description/robot.urdf.xacro (robot description, xacro)
@@ -3,5 +3,6 @@
     <!-- Example link -->
     <xacro:include filename="robot_core.xacro"/>
+    <xacro:include filename="properties.xacro"/>
+    <xacro:include filename="inertial_macros.xacro"/>
         <!-- Example link -->
-    <link name="base_link"></link>
 </robot>

Commit message: asdd

File: description/robot.urdf.xacro (robot description, xacro)
@@ -4,5 +4,5 @@
     <xacro:include filename="robot_core.xacro"/>
     <xacro:include filename="properties.xacro"/>
-    <xacro:include filename="inertial_macros.xacro"/>
-        <!-- Example link -->
+    <xacro:include filename="gazebo_control.xacro"/>
+    <!-- Example link -->
 </robot>

File: description/robot_core.xacro (robot description, xacro)
@@ -101,3 +101,17 @@
         </xacro:inertial_sphere>
     </link>
+    <gazebo reference="chassis">
+        <material>Gazebo/White</material>
+    </gazebo>
+    <gazebo reference="left_wheel">
+        <material>Gazebo/Blue</material>
+    </gazebo>
+    <gazebo reference="right_wheel">
+        <material>Gazebo/Blue</material>
+    </gazebo>
+    <gazebo reference="caster_wheel">
+        <material>Gazebo/Black</material>
+        <mu1 value = "0.001" />
+        <mu2 value = "0.001" />
+    </gazebo>
 </robot>

Commit message: test

File: description/robot.urdf.xacro (robot description, xacro)
@@ -4,4 +4,4 @@
     <xacro:include filename="robot_core.xacro"/>
         <!-- Example link -->
-    <link name="base_link"></link>
+    <link name="base_linkkk"></link>
 </robot>

Commit message: Class No.3

File: description/robot.urdf.xacro (robot description, xacro)
@@ -1,7 +1,9 @@
 <?xml version="1.0"?>
-<robot xmlns:xacro="http://www.ros.org/wiki/xacro"  name="robot">
+<robot xmlns:xacro="http://www.ros.org/wiki/xacro" name="robot">
     <!-- Example link -->
+    <xacro:include filename="properties.xacro"/>
     <xacro:include filename="robot_core.xacro"/>
-        <!-- Example link -->
-    <link name="base_linkkk"></link>
+    <xacro:include filename="inertial_macros.xacro"/>
+    <xacro:include filename="gazebo_control.xacro"/>
+    <xacro:include filename="lidar.xacro"/>
 </robot>

Commit message: Class4

File: description/robot.urdf.xacro (robot description, xacro)
@@ -4,6 +4,7 @@
     <xacro:include filename="robot_core.xacro"/>
     <xacro:include filename="properties.xacro"/>
-    <xacro:include filename="gazebo_control.xacro"/>
+     <!-- <xacro:include filename="gazebo_control.xacro"/>  -->
     <xacro:include filename="lidar.xacro"/>
+    <xacro:include filename="ros2_control.xacro"/>
     <!-- Example link -->
 </robot>

File: description/robot_core.xacro (robot description, xacro)
@@ -46,8 +46,8 @@
         </visual>
         <collision>
-            <geometry>
-                <cylinder radius="0.05" length="0.04"/>
-            </geometry>
-        </collision>
+	          <geometry>
+	              <sphere radius="0.05"/>
+	          </geometry>
+	      </collision>
         <xacro:inertial_cylinder mass="0.1" length="0.04" radius="0.05">
             <origin xyz="0 0 0" rpy="0 0 0"/>
@@ -71,5 +71,5 @@
         <collision>
             <geometry>
-                <cylinder radius="0.05" length="0.04"/>
+                <sphere radius="0.05" />
             </geometry>
         </collision>

Commit message: All

File: description/robot.urdf.xacro (robot description, xacro)
@@ -1,7 +1,10 @@
 <?xml version="1.0"?>
-<robot xmlns:xacro="http://www.ros.org/wiki/xacro">
+<robot xmlns:xacro="http://www.ros.org/wiki/xacro" name="my_bot">
     <!-- Example link -->
     <xacro:include filename="properties.xacro"/>
-    <xacro:include filename="robot_core.xacro"/>
+    <xacro:include filename="robot_core_ack.xacro"/>
     <xacro:include filename="inertial_macros.xacro"/>
+    <!--xacro:include filename="gazebo_control.xacro"/-->
+    <xacro:include filename="lidar.xacro"/>
+    <xacro:include filename="ros2_control_ack.xacro"/>
 </robot>

File: description/robot_core.xacro (robot description, xacro)
@@ -26,4 +26,7 @@
             </geometry>
         </collision>
+        <xacro:inertial_box mass="0.5" x="0.3" y="0.3" z="0.15">
+            <origin xyz="0.15 0 0.075" rpy="0 0 0"/>
+        </xacro:inertial_box>
     </link>
     <!-- left wheel joint -->
@@ -44,7 +47,10 @@
         <collision>
             <geometry>
-                <cylinder radius="0.05" length="0.04"/>
+                <sphere radius="0.05" />
             </geometry>
         </collision>
+        <xacro:inertial_cylinder mass="0.1" length="0.04" radius="0.05">
+            <origin xyz="0 0 0" rpy="0 0 0"/>
+        </xacro:inertial_cylinder>
     </link>
     <!-- right wheel joint -->
@@ -65,7 +71,10 @@
         <collision>
             <geometry>
-                <cylinder radius="0.05" length="0.04"/>
+                <sphere radius="0.05"/>
             </geometry>
         </collision>
+        <xacro:inertial_cylinder mass="0.1" length="0.04" radius="0.05">
+            <origin xyz="0 0 0" rpy="0 0 0"/>
+        </xacro:inertial_cylinder>
     </link>
     <!-- caster wheel joint -->
@@ -75,5 +84,5 @@
         <origin xyz="0.24 0 0"/>
     </joint>
-    <!-- left wheel link -->
+    <!-- caster wheel link -->
     <link name="caster_wheel">
         <visual>
@@ -88,4 +97,21 @@
             </geometry>
         </collision>
+        <xacro:inertial_sphere mass="0.1" radius="0.05">
+            <origin xyz="0 0 0" rpy="0 0 0"/>
+        </xacro:inertial_sphere>
     </link>
+    <gazebo reference="chassis">
+        <material>Gazebo/White</material>
+    </gazebo>
+    <gazebo reference="left_wheel">
+        <material>Gazebo/Blue</material>
+    </gazebo>
+    <gazebo reference="right_wheel">
+        <material>Gazebo/Blue</material>
+    </gazebo>
+    <gazebo reference="caster_wheel">
+        <material>Gazebo/Black</material>
+        <mu1 value = "0.001" />
+        <mu2 value = "0.001" />
+    </gazebo>
 </robot>

Commit message: Class No.5

File: description/robot.urdf.xacro (robot description, xacro)
@@ -5,5 +5,6 @@
     <xacro:include filename="robot_core.xacro"/>
     <xacro:include filename="inertial_macros.xacro"/>
-    <xacro:include filename="gazebo_control.xacro"/>
+    <xacro:include filename="ros2_control.xacro"/>
+    <!--xacro:include filename="gazebo_control.xacro"/ -->
     <xacro:include filename="lidar.xacro"/>
 </robot>

File: description/robot_core.xacro (robot description, xacro)
@@ -47,5 +47,5 @@
         <collision>
             <geometry>
-                <cylinder radius="0.05" length="0.04"/>
+                <sphere radius="0.05" />
             </geometry>
         </collision>
@@ -71,5 +71,5 @@
         <collision>
             <geometry>
-                <cylinder radius="0.05" length="0.04"/>
+                <sphere radius="0.05"/>
             </geometry>
         </collision>
@@ -84,5 +84,5 @@
         <origin xyz="0.24 0 0"/>
     </joint>
-    <!-- left wheel link -->
+    <!-- caster wheel link -->
     <link name="caster_wheel">
         <visual>
@@ -101,5 +101,4 @@
         </xacro:inertial_sphere>
     </link>
-    <!-- Gazebo  -->
     <gazebo reference="chassis">
         <material>Gazebo/White</material>
