Commit message: sebas Branch

File: description/lidar.xacro (robot description, xacro)
@@ -5,5 +5,5 @@
         <parent link="chassis"/>
         <child link="laser_frame"/>
-        <origin xyz="0.1 0 0.175" rpy="0 0 0"/>
+        <origin xyz="0.1 0 0.11" rpy="0 0 0"/>
     </joint>
     <!-- laser_frame -->

Commit message: Added twist mux

File: description/lidar.xacro (robot description, xacro)
@@ -5,5 +5,5 @@
         <parent link="chassis"/>
         <child link="laser_frame"/>
-        <origin xyz="0.1 0 0.11" rpy="0 0 0"/>
+        <origin xyz="0.1 0 0.1" rpy="0 0 0"/>
     </joint>
     <!-- laser_frame -->

File: description/robot_core_ack.xacro (robot description, xacro)
@@ -219,26 +219,26 @@
     <gazebo reference="chassis">
         <material>Gazebo/White</material>
-        <mu1 value = "0.1" />
-        <mu2 value = "0.1" />
+        <mu1 value = "0.3" />
+        <mu2 value = "0.3" />
     </gazebo>
     <gazebo reference="rear_left_wheel">
         <material>Gazebo/Blue</material>
-        <mu1 value = "0.1" />
-        <mu2 value = "0.1" />
+        <mu1 value = "0.3" />
+        <mu2 value = "0.3" />
     </gazebo>
     <gazebo reference="rear_right_wheel">
         <material>Gazebo/Blue</material>
-         <mu1 value = "0.1" />
-        <mu2 value = "0.1" />
+         <mu1 value = "0.3" />
+        <mu2 value = "0.3" />
     </gazebo>
      <gazebo reference="front_left_wheel">
         <material>Gazebo/Blue</material>
-         <mu1 value = "0.1" />
-        <mu2 value = "0.1" />
+         <mu1 value = "0.3" />
+        <mu2 value = "0.3" />
     </gazebo>
     <gazebo reference="front_right_wheel">
         <material>Gazebo/Blue</material>
-         <mu1 value = "0.02" />
-        <mu2 value = "0.02" />
+         <mu1 value = "0.3" />
+        <mu2 value = "0.3" />
     </gazebo>
     <gazebo reference="right_steering_link">
